Commit message: controller, camera simulation completed

File: robot_model/urdf/my_robot.urdf (robot description, URDF)
Before this commit: robot adobe, 9 links, 8 joints
Links:
- link base_link: geometry collision mesh filename=package://robot_model/meshes/base_link_collision.STL; visual mesh filename=package://robot_model/meshes/base_link.STL

Commit message: Update

File: robot_model/urdf/my_robot.urdf (robot description, URDF)
Before this commit: robot adobe, 9 links, 8 joints
Links:
- removed link camera_link
- removed link lidar_link
- link base_link: mass 0.61219 -> 0.70318
- link pitch_b_link: mass 0.0025724 -> 0.011494
- link roll_b_link: mass 0.0025724 -> 0.011494
- link yaw_b_link: mass 0.0025724 -> 0.011494
Joints:
- removed joint camera_joint
- removed joint lidar_joint
- joint lw_joint: origin xyz=-0.032594 0.05077 0.01125 rpy=1.5708 -0.0050356 -3.1329 -> xyz=-0.069392 0.090498 0.01125 rpy=1.5708 0.0050356 0.00872
- joint roll_b_joint: origin xyz=0.073997 0.00064527 -0.014 rpy=0 0 0 -> xyz=0.064998 0.00056679 -0.009 rpy=0 0 0
- joint rw_joint: origin xyz=-0.031704 -0.05133 0.01125 rpy=1.5708 -0.0050356 -3.1329 -> xyz=-0.067803 -0.091695 0.01125 rpy=1.5708 0.0050356 0.00872
